Commit message: feat: add third target

File: mani_skill/assets/robots/xarm6/xarm6_robotiq.urdf (robot description, URDF)
Before this commit: robot xarm6, 21 links, 20 joints
Links:
- added link ego_camera_link
Joints:
- added joint ego_camera_link_joint: type fixed, parent link6, child ego_camera_link, origin xyz=0.0675 0.0115 -0.016315 rpy=3.141592653589793 0.0 0.0
